Commit message: added moveit2 functionality

File: install/tentacle_description/share/tentacle_description/urdf/tentacle.xacro (robot description, xacro)
@@ -6,4 +6,5 @@
   <xacro:include filename="$(find tentacle_description)/urdf/tentacle_gazebo.xacro"/>
   <xacro:include filename="$(find tentacle_description)/urdf/tentacle_ros2_control.xacro" />
+  <link name="world"/>
   <link name="base_link">
   <inertial>
@@ -146,4 +147,9 @@
   </collision>
 </link>
+<joint name="virtual_joint" type="fixed">
+  <parent link="world"/>
+  <child link="base_link"/>
+  <origin xyz="0 0 0" rpy="0 0 0"/>
+</joint>
 <joint name="Revolute_1" type="continuous">
   <origin xyz="0.003249 0.000454 0.035" rpy="0 0 0"/>
@@ -157,5 +163,5 @@
   <child link="forearm_1"/>
   <axis xyz="0.0 -1.0 0.0"/>
-  <limit upper="0.0" lower="-2.541593" effort="100" velocity="100"/>
+  <limit upper="0.1" lower="-2.541593" effort="100" velocity="100"/>
 </joint>
 <joint name="Revolute_3" type="revolute">
@@ -164,5 +170,5 @@
   <child link="arm_1"/>
   <axis xyz="-0.0 1.0 -0.0"/>
-  <limit upper="0.0" lower="-3.141593" effort="100" velocity="100"/>
+  <limit upper="0.1" lower="-3.141593" effort="100" velocity="100"/>
 </joint>
 <joint name="Rigid" type="fixed">

File: install/tentacle_description/share/tentacle_description/urdf/tentacle_ros2_control.xacro (robot description, xacro)
@@ -22,5 +22,5 @@
             <command_interface name="position">
                 <param name="min">-2.541593</param>
-                <param name="max">0.0</param>
+                <param name="max">0.1</param>
             </command_interface>
             <state_interface name="position"/>
@@ -29,5 +29,5 @@
             <command_interface name="position">
                 <param name="min">-3.141593</param>
-                <param name="max">0.0</param>
+                <param name="max">0.1</param>
             </command_interface>
             <state_interface name="position"/>
